File: pcb/mcu-adapter/tC-mcu-adapter-rev1.brd (EAGLE design)
At the start: 27.6 x 58.2 mm, 35 parts, among them CN1 FPC_CONN_18PIN_0.5MM_SMT, U1 CY8C5XXX-68-N, U2 STM8L051F3P6, U3 4052D

Commit message: Minor tweaks to MCU adapter board
- Cleaned up schematic view
- Finished CapSense breakout pads to second board
- Changed caps to 0603 to ease hand soldering
- Minor stuff to silkscreen.
Parts:
- added CSD: CAP_INTERCONNECT, _dc801:CAP_INTERCONNECT
- C10, C11, C12, C2, C3, C4, C5, C6, C7, C8, C9: device rcl:C0402K -> rcl:C0603K
- moved C11 0.64 mm to (8.33, 15.2)
- moved C12 0.64 mm to (8.33, 13.7)
- moved C4 0.64 mm to (14.6, 12.1)
- moved C5 0.64 mm to (14.6, 13.7)
- moved C7 0.64 mm to (8.33, 12.1)
- moved C8 0.64 mm to (14.6, 15.2)
- moved C9 0.31 mm to (13.8, 8.18)
- moved SWIM 0.27 mm to (23.7, 52.7), flipped to the bottom
- moved LED3 0.25 mm to (26.4, 32.3)
- moved LED7 0.25 mm to (26.4, 36.3)
- moved R1 0.25 mm to (10.4, 35.1)
- moved A1 0.25 mm to (11.4, 31.5)
- moved C1 0.25 mm to (12.2, 22.0)
- moved U1 0.25 mm to (11.4, 11.9)
- moved L1 0.25 mm to (17.3, 1.98)
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Connections:
- net CSD_B0: now also CSD.1
- net CSD_B1: now also CSD.2
- net CSD_B2: now also CSD.3
- net CSD_B3: now also CSD.4
Routing:
- net CSD_B0: track 32.4 -> 21.2 mm, vias 0 -> 1
- net CSD_B1: track 31.7 -> 22.4 mm, vias 0 -> 1
- net CSD_B2: track 29.7 -> 22.5 mm, vias 0 -> 1
- net CSD_B3: track 29.1 -> 23.9 mm, vias 0 -> 1
- net +3V3: track 160.6 -> 162.2 mm
- net GND: track 115.6 -> 114.2 mm
- net CMOD: track 4.44 -> 5.55 mm
- net XBEE_RST: track 29.5 -> 28.6 mm
- net ST_SWIM: track 28.6 -> 29.3 mm
- net VCCA: track 2.97 -> 2.39 mm
