File: pcb/mcu-adapter/tC-mcu-adapter-rev1.sch (EAGLE design)
At the start: 35 parts, among them CN1 FPC_CONN_18PIN_0.5MM_SMT, U1 CY8C5XXX-68-N, U2 STM8L051F3P6, U3 4052D

Commit message: Minor tweaks to MCU adapter board
- Cleaned up schematic view
- Finished CapSense breakout pads to second board
- Changed caps to 0603 to ease hand soldering
- Minor stuff to silkscreen.
Parts:
- added CSD: CAP_INTERCONNECT, _dc801:CAP_INTERCONNECT
- C10, C11, C12, C2, C3, C4, C5, C6, C7, C8, C9: device rcl:C-EUC0402K -> rcl:C-EUC0603K
Connections:
- net CSD_B0: now also CSD.1
- net CSD_B1: now also CSD.2
- net CSD_B2: now also CSD.3
- net CSD_B3: now also CSD.4
Other:
- note added: "CapSense"
- note added: "LED PWM and Serial Mux Selector MCU"
- note added: "Main MCU"
- note added: "Serial Mux"
- note added: "Socket Interface"
- note added: "To Breakout"
- note added: "User GPIO"
- note added: "User LEDs"
- moved on the sheet: A1, C1, C10, C11, C12, C13, C14, C2, C3, C4, C5, C6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
